File: Rev_B/KiCad_PCB_Files/AI_Board_Rev_B.kicad_pcb (KiCad board)
At the start: 2 copper layers, 130 x 165 mm, 49 parts, among them J1 DC37_Socket_MountingHoles, J10 AI4 M12, J11 AI4 XT30, J12 AI5 M12, J13 AI5 XT30, J14 AI6 M12, J15 AI6 XT30, J16 AI7 M12, J17 AI7 XT30, J18 AI8 M12, J19 AI8 XT30, J2 AI0 M12, J20 AI9 M12, J21 AI9 XT30, J22 AI10 M12, J23 AI10 XT30, J24 AI11 M12, J25 AI11 XT30, J26 AI12 M12, J27 AI12 XT30, J28 AI13 M12, J29 AI13 XT30, J3 AI0 XT30, J30 AI14 M12, J31 AI14 XT30, J32 AI15 M12, J33 AI15 XT30, J4 AI1 M12, J5 AI1 XT30, J6 AI2 M12, J7 AI2 XT30, J8 AI3 M12, J9 AI3 XT30

Commit message: Add files via upload
Routing:
- net /AI10+: track 136.3 -> 133.1 mm

Commit message: Add files via upload
Other:
- board text added: "SINE LABORE NIHIL PER ARDUA AD ALTA"

Commit message: Add files via upload
Parts:
- added G***: LOGO, MST RDT PR:MSTRDTLogoFootprint11mm, F.Cu at (30.0, 155.0)
- added M3: MountingHole_3.2mm_M3, MountingHole:MountingHole_3.2mm_M3, F.Cu at (20.0, 20.0)
- added M3: MountingHole_3.2mm_M3, MountingHole:MountingHole_3.2mm_M3, F.Cu at (140.0, 20.0)
- added M3: MountingHole_3.2mm_M3, MountingHole:MountingHole_3.2mm_M3, F.Cu at (20.0, 175.0)
- added M3: MountingHole_3.2mm_M3, MountingHole:MountingHole_3.2mm_M3, F.Cu at (140.0, 175.0)
Other:
- board text added: "AI0"
- board text added: "AI1"
- board text added: "AI10"
- board text added: "AI11"
- board text added: "AI12"
- board text added: "AI13"
- board text added: "AI14"
- board text added: "AI15"
- board text added: "AI2"
- board text added: "AI3"
- board text added: "AI4"
- board text added: "AI5"
- board text added: "AI6"
- board text added: "AI7"
- board text added: "AI8"
- board text added: "AI9"
